File: pcb/rs485-lowpower.kicad_pcb (KiCad board)
At the start: 2 copper layers, 45.4 x 31.7 mm, 16 parts, among them U4 MAX487

Commit message: reupload pcb file
Parts:
- removed RS485-UBBLPV1.0: 282837-4, TE_282837-4
- added RS485-UGMLPV1.0: 282837-4, TE_282837-4, F.Cu at (151.2, 114.5)
- added U$1: ID000015, CERT-SMALL-SILK, F.Cu at (133.8, 110.2)
- U4: value MAX487 -> MAX485CSA+T
Routing:
- net VCC: track 137.1 -> 140.1 mm, vias 3 -> 4
